File: KiCad/VCO_RPIpico.kicad_pcb (KiCad board)
At the start: 2 copper layers, 138 x 83 mm, 81 parts, among them J1 AudioJack3_Ground, J2 Power Jack, SW1 LFO1/2, SW2 Select LFO WaveForm, SW3 Fire4, SW4 Fire3, SW5 Fire2, SW6 Fire1, SW7 Shift2/Save, SW8 Shift1 / Select Bank, U2 PT2399, U3 L7805

Commit message: Display
Parts:
- added C25: 1µ, Capacitor_SMD:CP_Elec_4x5.7, F.Cu at (200.0, 106.6)
- added Q1: 2N7002, Package_TO_SOT_SMD:SOT-23, F.Cu at (215.8, 85.3)
- added R31: 10k, Resistor_SMD:R_1206_3216Metric, F.Cu at (210.6, 84.7)
- added U1: ER_OLEDM0.91_1x-I2C, Display:Adafruit_SSD1306, F.Cu at (205.8, 119.1)
- C17, C18: footprint Capacitor_Tantalum_SMD:CP_EIA-2012-12_Kemet-R_Pad1.30x1.05mm_HandSolder -> Capacitor_SMD:CP_Elec_4x5.7
Connections:
- A1 pad 1: unconnected-(A1-GPIO0-Pad1) -> Net-(A1-GPIO0)
- A1 pad 2: unconnected-(A1-GPIO1-Pad2)_1 -> Net-(A1-GPIO1)
- A1 pad 29: unconnected-(A1-GPIO22-Pad29)_1 -> /mute
